Commit message: serial communication with stm

File: description/robot_core.xacro (robot description, xacro)
@@ -40,5 +40,5 @@
             <cylinder length="0.025" radius="0.03" />
         </geometry>
-        <material name="blue"/>
+        <material name="silver"/>
     </visual>
     <collision>
@@ -46,5 +46,5 @@
             <cylinder length="0.025" radius="0.03" />
         </geometry>
-        <material name="blue"/>
+        <material name="silver"/>
     </collision>
 </link>
@@ -60,5 +60,5 @@
             <cylinder length="0.025" radius="0.03" />
         </geometry>
-        <material name="blue"/>
+        <material name="silver"/>
     </visual>
     <collision>
@@ -66,5 +66,5 @@
             <cylinder length="0.025" radius="0.03" />
         </geometry>
-        <material name="blue"/>
+        <material name="silver"/>
     </collision>
 </link>
@@ -80,5 +80,5 @@
             <cylinder length="0.025" radius="0.03" />
         </geometry>
-        <material name="blue"/>
+        <material name="silver"/>
     </visual>
     <collision>
@@ -86,5 +86,5 @@
             <cylinder length="0.025" radius="0.03" />
         </geometry>
-        <material name="blue"/>
+        <material name="silver"/>
     </collision>
 </link>
@@ -100,5 +100,5 @@
             <cylinder length="0.025" radius="0.03" />
         </geometry>
-        <material name="blue"/>
+        <material name="silver"/>
     </visual>
     <collision>
@@ -106,5 +106,5 @@
             <cylinder length="0.025" radius="0.03" />
         </geometry>
-        <material name="blue"/>
+        <material name="silver"/>
     </collision>
 </link>

Commit message: odometry rotating on the rviz, encoders not implemented

File: description/robot_core.xacro (robot description, xacro)
@@ -3,4 +3,10 @@
 <xacro:include filename="materials.xacro" />
 <xacro:include filename="inertial_macros.xacro" />
+<joint name="odom" type="fixed">
+  <parent link="odom"/>
+  <child link="base_link"/>
+  <origin xyz="0 0 0" rpy="0 0 0"/>
+</joint>
+<link name="odom"/>
 <link name="base_link">
 </link>
