Commit message: initial lidar node

File: description/materials.xacro (robot description, xacro)
@@ -4,3 +4,6 @@
     <color rgba="0.700 0.700 0.700 1.000"/>
   </material>
+  <material name="red">
+    <color rgba="1 0 0 1"/>
+  </material>
 </robot>

File: description/robot_core.xacro (robot description, xacro)
@@ -3,4 +3,5 @@
 <xacro:include filename="materials.xacro" />
 <xacro:include filename="inertial_macros.xacro" />
+<xacro:include filename="lidar.xacro" />
 <joint name="odom" type="fixed">
   <parent link="odom"/>
